File: Transformerless Power Supply/transformerless power supply/transformerless power supply.kicad_sch (KiCad schematic)
At the start: 18 parts, among them J1 Screw_Terminal_01x02, J2 Screw_Terminal_01x02, U1 LM7805_TO220

Commit message: kicad files
Parts:
- C1: footprint (none) -> Capacitor_THT:C_Disc_D4.7mm_W2.5mm_P5.00mm
- C2, C3: footprint (none) -> Capacitor_THT:CP_Radial_D10.0mm_P5.00mm
- C4: footprint (none) -> Capacitor_THT:C_Rect_L18.0mm_W6.0mm_P15.00mm_FKS3_FKP3
- D5, D6: footprint (none) -> Diode_THT:D_A-405_P7.62mm_Horizontal
- D7: renamed from D?; footprint (none) -> LED_THT:LED_D5.0mm
- J1, J2: footprint (none) -> TerminalBlock:TerminalBlock_MaiXu_MX126-5.0-02P_1x02_P5.00mm
- R1, R2, R3, R4: footprint (none) -> Resistor_THT:R_Axial_DIN0207_L6.3mm_D2.5mm_P7.62mm_Horizontal
Connections:
- net GND: now reaches C1.2, C2.2, C3.2, D2.2 (A), D4.2 (A), D7.1 (K), J2.2 (Pin_2), R1.2, R2.2, U1.2 (GND)
- net 5V: now reaches C3.1, J2.1 (Pin_1), U1.3 (VO)
